File: Circuito/Burbujas.kicad_sch (KiCad schematic)
At the start: 19 parts, among them J1 Bornera x 2, J2 Bornera x 3, J3 Bornera x 2, J4 Bornera x 2, SW1 tact switch, SW2 tact switch, SW3 tact switch, SW4 tact switch, U1 LM7805_TO220, U2 PIC12F629-IP

Commit message: Correcciones
Correcciones
Connections:
- net at R1.2, SW3.2: now also U2.4 (GP3); no longer U2.5 (GP2)
- net at R2.1: now also U2.7 (GP0); no longer U2.4 (GP3)
- net at R3.1: now also U2.6 (GP1); no longer U2.3 (GP4)
- net at SW1.2: now also U2.2 (GP5); no longer U2.7 (GP0)
- net at SW2.2: now also U2.3 (GP4); no longer U2.6 (GP1)
- net at SW4.2: now also U2.5 (GP2); no longer U2.2 (GP5)
Changed lines of the file:
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@@
   (junction (at 110.49 165.1) (diameter 0) (color 0 0 0 0)
   )
-  (junction (at 105.41 73.66) (diameter 0) (color 0 0 0 0)
-  )
   (junction (at 120.65 154.94) (diameter 0) (color 0 0 0 0)
   )
+  (junction (at 105.41 68.58) (diameter 0) (color 0 0 0 0)
+  )
   (junction (at 81.28 81.28) (diameter 0) (color 0 0 0 0)
   )
@@
     (stroke (width 0) (type default) (color 0 0 0 0))
   )
+  (wire (pts (xy 102.87 71.12) (xy 102.87 74.93))
+    (stroke (width 0) (type default) (color 0 0 0 0))
+  )
   (wire (pts (xy 120.65 165.1) (xy 120.65 163.83))
     (stroke (width 0) (type default) (color 0 0 0 0))
   )
+  (wire (pts (xy 147.32 68.58) (xy 163.83 68.58))
+    (stroke (width 0) (type default) (color 0 0 0 0))
+  )
   (wire (pts (xy 78.74 165.1) (xy 88.9 165.1))
     (stroke (width 0) (type default) (color 0 0 0 0))
   )
+  (wire (pts (xy 102.87 74.93) (xy 92.71 74.93))
+    (stroke (width 0) (type default) (color 0 0 0 0))
+  )
   (wire (pts (xy 180.34 76.2) (xy 180.34 106.68))
     (stroke (width 0) (type default) (color 0 0 0 0))
   )
-  (wire (pts (xy 92.71 68.58) (xy 116.84 68.58))
-    (stroke (width 0) (type default) (color 0 0 0 0))
-  )
-  (wire (pts (xy 92.71 87.63) (xy 105.41 87.63))
+  (wire (pts (xy 147.32 71.12) (xy 156.21 71.12))
+    (stroke (width 0) (type default) (color 0 0 0 0))
+  )
+  (wire (pts (xy 156.21 71.12) (xy 156.21 76.2))
     (stroke (width 0) (type default) (color 0 0 0 0))
   )
@@
     (stroke (width 0) (type default) (color 0 0 0 0))
   )
-  (wire (pts (xy 105.41 87.63) (xy 105.41 91.44))
+  (wire (pts (xy 92.71 68.58) (xy 100.33 68.58))
     (stroke (width 0) (type default) (color 0 0 0 0))
   )
@@
     (stroke (width 0) (type default) (color 0 0 0 0))
   )
-  (wire (pts (xy 147.32 73.66) (xy 149.86 73.66))
+  (wire (pts (xy 105.41 81.28) (xy 92.71 81.28))
     (stroke (width 0) (type default) (color 0 0 0 0))
   )
@@
     (stroke (width 0) (type default) (color 0 0 0 0))
   )
+  (wire (pts (xy 100.33 73.66) (xy 116.84 73.66))
+    (stroke (width 0) (type default) (color 0 0 0 0))
+  )
   (wire (pts (xy 180.34 68.58) (xy 180.34 55.88))
     (stroke (width 0) (type default) (color 0 0 0 0))
   )
-  (wire (pts (xy 100.33 71.12) (xy 100.33 74.93))
+  (wire (pts (xy 148.59 73.66) (xy 148.59 92.71))
     (stroke (width 0) (type default) (color 0 0 0 0))
   )
@@
     (stroke (width 0) (type default) (color 0 0 0 0))
   )
-  (wire (pts (xy 105.41 81.28) (xy 92.71 81.28))
+  (wire (pts (xy 116.84 68.58) (xy 105.41 68.58))
     (stroke (width 0) (type default) (color 0 0 0 0))
   )
@@
     (stroke (width 0) (type default) (color 0 0 0 0))
   )
-  (wire (pts (xy 105.41 64.77) (xy 105.41 73.66))
+  (wire (pts (xy 105.41 68.58) (xy 105.41 81.28))
     (stroke (width 0) (type default) (color 0 0 0 0))
   )
@@
     (stroke (width 0) (type default) (color 0 0 0 0))
   )
-  (wire (pts (xy 105.41 73.66) (xy 105.41 81.28))
-    (stroke (width 0) (type default) (color 0 0 0 0))
-  )
-  (wire (pts (xy 116.84 71.12) (xy 100.33 71.12))
-    (stroke (width 0) (type default) (color 0 0 0 0))
-  )
   (wire (pts (xy 67.31 154.94) (xy 69.85 154.94))
     (stroke (width 0) (type default) (color 0 0 0 0))
   )
+  (wire (pts (xy 100.33 68.58) (xy 100.33 73.66))
+    (stroke (width 0) (type default) (color 0 0 0 0))
+  )
   (wire (pts (xy 105.41 52.07) (xy 132.08 52.07))
     (stroke (width 0) (type default) (color 0 0 0 0))
@@
     (stroke (width 0) (type default) (color 0 0 0 0))
   )
+  (wire (pts (xy 105.41 87.63) (xy 92.71 87.63))
+    (stroke (width 0) (type default) (color 0 0 0 0))
+  )
   (wire (pts (xy 110.49 154.94) (xy 120.65 154.94))
     (stroke (width 0) (type default) (color 0 0 0 0))
@@
     (stroke (width 0) (type default) (color 0 0 0 0))
   )
-  (wire (pts (xy 100.33 74.93) (xy 92.71 74.93))
+  (wire (pts (xy 156.21 76.2) (xy 163.83 76.2))
     (stroke (width 0) (type default) (color 0 0 0 0))
   )
@@
     (stroke (width 0) (type default) (color 0 0 0 0))
   )
-  (wire (pts (xy 147.32 71.12) (xy 156.21 71.12))
-    (stroke (width 0) (type default) (color 0 0 0 0))
-  )
-  (wire (pts (xy 149.86 91.44) (xy 105.41 91.44))
+  (wire (pts (xy 105.41 92.71) (xy 105.41 87.63))
     (stroke (width 0) (type default) (color 0 0 0 0))
   )
@@
     (stroke (width 0) (type default) (color 0 0 0 0))
   )
-  (wire (pts (xy 147.32 68.58) (xy 163.83 68.58))
-    (stroke (width 0) (type default) (color 0 0 0 0))
-  )
-  (wire (pts (xy 156.21 71.12) (xy 156.21 76.2))
-    (stroke (width 0) (type default) (color 0 0 0 0))
-  )
-  (wire (pts (xy 156.21 76.2) (xy 163.83 76.2))
-    (stroke (width 0) (type default) (color 0 0 0 0))
-  )
   (wire (pts (xy 120.65 154.94) (xy 120.65 153.67))
     (stroke (width 0) (type default) (color 0 0 0 0))
@@
     (stroke (width 0) (type default) (color 0 0 0 0))
   )
+  (wire (pts (xy 147.32 73.66) (xy 148.59 73.66))
+    (stroke (width 0) (type default) (color 0 0 0 0))
+  )
   (wire (pts (xy 191.77 101.6) (xy 191.77 96.52))
     (stroke (width 0) (type default) (color 0 0 0 0))
   )
-  (wire (pts (xy 116.84 73.66) (xy 105.41 73.66))
-    (stroke (width 0) (type default) (color 0 0 0 0))
-  )
   (wire (pts (xy 88.9 165.1) (xy 101.6 165.1))
     (stroke (width 0) (type default) (color 0 0 0 0))
@@
     (stroke (width 0) (type default) (color 0 0 0 0))
   )
-  (wire (pts (xy 149.86 73.66) (xy 149.86 91.44))
-    (stroke (width 0) (type default) (color 0 0 0 0))
-  )
   (wire (pts (xy 193.04 58.42) (xy 193.04 59.69))
     (stroke (width 0) (type default) (color 0 0 0 0))
@@
   )
   (wire (pts (xy 81.28 68.58) (xy 81.28 74.93))
+    (stroke (width 0) (type default) (color 0 0 0 0))
+  )
+  (wire (pts (xy 148.59 92.71) (xy 105.41 92.71))
+    (stroke (width 0) (type default) (color 0 0 0 0))
+  )
+  (wire (pts (xy 105.41 68.58) (xy 105.41 64.77))
+    (stroke (width 0) (type default) (color 0 0 0 0))
+  )
+  (wire (pts (xy 116.84 71.12) (xy 102.87 71.12))
     (stroke (width 0) (type default) (color 0 0 0 0))
   )
@@
     (pin "1")
   )
-  (symbol (lib_id "MCU_Microchip_PIC12:PIC12F629-IP") (at 132.08 71.12 0) (unit 1)
-    (in_bom yes) (on_board yes) (fields_autoplaced)
-    (property "Reference" "U2" (id 0) (at 134.0994 55.88 0)
-      (effects (font (size 1.27 1.27)) (justify left))
-    )
-    (property "Value" "PIC12F629-IP" (id 1) (at 134.0994 58.42 0)
-      (effects (font (size 1.27 1.27)) (justify left))
-    )
-    (property "Footprint" "Package_DIP:DIP-8_W7.62mm" (id 2) (at 147.32 54.61 0)
-      (effects (font (size 1.27 1.27)) hide)
-    )
+  (symbol (lib_id "MCU_Microchip_PIC12:PIC12F629-IP") (at 132.08 71.12 0) (mirror y) (unit 1)
+    (in_bom yes) (on_board yes) (fields_autoplaced)
+    (property "Reference" "U2" (id 0) (at 132.6006 55.88 0)
+      (effects (font (size 1.27 1.27)) (justify right))
+    )
+    (property "Value" "PIC12F629-IP" (id 1) (at 132.6006 58.42 0)
+      (effects (font (size 1.27 1.27)) (justify right))
+    )
+    (property "Footprint" "Package_DIP:DIP-8_W7.62mm" (id 2) (at 116.84 54.61 0)
+      (effects (font (size 1.27 1.27)) hide)
+    )
